Commit message: localizacao

File: src/simu/urdf/robot.urdf.xacro (robot description, xacro)
@@ -2,11 +2,11 @@
 <robot name="my_robot" xmlns:xacro="http://www.ros.org/wiki/xacro">
   <!--=========================== PLUGINS ===========================-->
-  <xacro:include filename="$(find simu)/urdf/robot.gazebo.xacro" />
+  <xacro:include filename="$(find robot_description)/urdf/robot.gazebo.xacro" />
   <!--=========================== ROBOT PARTS ===========================-->
-  <xacro:include filename="$(find simu)/urdf/robot_parts/carcaca.xacro" />
-  <xacro:include filename="$(find simu)/urdf/robot_parts/traction_wheel.xacro" />
-  <xacro:include filename="$(find simu)/urdf/robot_parts/tray.xacro" />
-  <xacro:include filename="$(find simu)/urdf/robot_parts/piston.xacro" />
-  <xacro:include filename="$(find simu)/urdf/robot_parts/omni_wheel.xacro" />
+  <xacro:include filename="$(find robot_description)/urdf/robot_parts/carcaca.xacro" />
+  <xacro:include filename="$(find robot_description)/urdf/robot_parts/traction_wheel.xacro" />
+  <xacro:include filename="$(find robot_description)/urdf/robot_parts/tray.xacro" />
+  <xacro:include filename="$(find robot_description)/urdf/robot_parts/piston.xacro" />
+  <xacro:include filename="$(find robot_description)/urdf/robot_parts/omni_wheel.xacro" />
   <!--=========================== SENSORS ===========================-->
   <xacro:arg name="sensor_imu" default="true" />
@@ -15,14 +15,14 @@
   <xacro:arg name="sensor_camera" default="true" />
   <xacro:if value="$(arg sensor_imu)">
-    <xacro:include filename="$(find simu)/urdf/sensors/imu.xacro" />
+    <xacro:include filename="$(find robot_description)/urdf/sensors/imu.xacro" />
   </xacro:if>
   <xacro:if value="$(arg sensor_lidar)">
-    <xacro:include filename="$(find simu)/urdf/sensors/lidar.xacro" />
+    <xacro:include filename="$(find robot_description)/urdf/sensors/lidar.xacro" />
   </xacro:if>
   <xacro:if value="$(arg sensor_rplidar)">
-    <xacro:include filename="$(find simu)/urdf/sensors/rplidar.xacro" />
+    <xacro:include filename="$(find robot_description)/urdf/sensors/rplidar.xacro" />
   </xacro:if>
   <xacro:if value="$(arg sensor_camera)">
-    <xacro:include filename="$(find simu)/urdf/sensors/camera.xacro" />
+    <xacro:include filename="$(find robot_description)/urdf/sensors/camera.xacro" />
   </xacro:if>
 </robot>

File: src/simu/urdf/robot_parts/carcaca.xacro (robot description, xacro)
@@ -6,18 +6,20 @@
             <mu1 value="0.3" />
             <mu2 value="0.3" />
-            <kp value="10000000.0" />
-            <kd value="1000" />
+            <kp value="1000000.0" />
+            <kd value="100" />
             <fdir1 value="0 0 0" />
         </gazebo>
         <link name="${base_link}">
             <inertial>
-                <mass value="15" />
+                <mass value="2.4" />
                 <origin rpy="0  0  3.14" xyz="0  0  0.0118" />
-                <inertia ixx="1" ixy="0" ixz="0" iyy="1" iyz="0" izz="1" />
+                <inertia ixx="0.019995" ixy="0.0" ixz="0.0"
+                iyy="0.019995" iyz="0.0"
+                izz="0.03675" />
             </inertial>
             <collision name="${base_link}_collision">
                 <origin rpy="0  0  3.14" xyz="0  0  0.0118" />
                 <geometry>
-                    <mesh filename="package://simu/models/laser_robot/meshes/carcaca.dae" scale="1 1 1" />
+                    <mesh filename="package://robot_description/models/laser_robot/meshes/carcaca.dae" scale="1 1 1" />
                 </geometry>
             </collision>
@@ -25,5 +27,5 @@
                 <origin rpy="0  0  3.14" xyz="0  0  0.0118" />
                 <geometry>
-                    <mesh filename="package://simu/models/laser_robot/meshes/carcaca.dae" scale="1 1 1" />
+                    <mesh filename="package://robot_description/models/laser_robot/meshes/carcaca.dae" scale="1 1 1" />
                 </geometry>
             </visual>

File: src/simu/urdf/robot_parts/omni_wheel.xacro (robot description, xacro)
@@ -24,5 +24,5 @@
                 <origin rpy="0 0 0" xyz="0 0 0" />
                 <geometry>
-                    <mesh filename="package://simu/models/laser_robot/omni_wheel/meshes/roda_omni.obj" scale="1 1 1" />
+                    <mesh filename="package://robot_description/models/laser_robot/omni_wheel/meshes/roda_omni.obj" scale="1 1 1" />
                 </geometry>
             </collision>
@@ -30,5 +30,5 @@
                 <origin rpy="0 0 0" xyz="0 0 0" />
                 <geometry>
-                    <mesh filename="package://simu/models/laser_robot/omni_wheel/meshes/roda_omni.obj" scale="1 1 1" />
+                    <mesh filename="package://robot_description/models/laser_robot/omni_wheel/meshes/roda_omni.obj" scale="1 1 1" />
                 </geometry>
             </visual>

File: src/simu/urdf/robot_parts/piston.xacro (robot description, xacro)
@@ -27,5 +27,5 @@
                 <origin rpy="0  0  0" xyz="0 0 0" />
                 <geometry>
-                    <mesh filename="package://simu/models/laser_robot/meshes/piston.dae" scale="1 1 1" />
+                    <mesh filename="package://robot_description/models/laser_robot/meshes/piston.dae" scale="1 1 1" />
                 </geometry>
             </collision>
@@ -33,5 +33,5 @@
                 <origin rpy="0  0  0" xyz="0 0 0" />
                 <geometry>
-                    <mesh filename="package://simu/models/laser_robot/meshes/piston.dae" scale="1 1 1" />
+                    <mesh filename="package://robot_description/models/laser_robot/meshes/piston.dae" scale="1 1 1" />
                 </geometry>
             </visual>

File: src/simu/urdf/robot_parts/traction_wheel.xacro (robot description, xacro)
@@ -11,8 +11,10 @@
         <gazebo reference="${prefix}">
             <selfCollide>false</selfCollide>
-            <mu1 value="100" />
-            <mu2 value="50" />
-            <kp value="10000000.0" />
-            <kd value="1000" />
+            <mu1>1.0</mu1>
+            <mu2>1.0</mu2>
+            <kp>1000000.0</kp>
+            <kd>100.0</kd>
+            <minDepth>0.001</minDepth>
+            <maxVel>1.0</maxVel>
             <fdir1 value="0 0 0" />
         </gazebo>
@@ -21,10 +23,12 @@
                 <mass value="1" />
                 <origin rpy="0 0 0" xyz="0 0 0" />
-                <inertia ixx="1" ixy="0" ixz="0" iyy="1" iyz="0" izz="1" />
+                <inertia ixx="0.001" ixy="0.0" ixz="0.0"
+                iyy="0.001" iyz="0.0"
+                izz="0.001" />
             </inertial>
             <collision name="${prefix}_collision">
                 <origin rpy="0 0 0" xyz="0 0 0" />
                 <geometry>
-                    <mesh filename="package://simu/models/laser_robot/wheel/meshes/roda.obj" scale="1 1 1" />
+                    <mesh filename="package://robot_description/models/laser_robot/wheel/meshes/roda.obj" scale="1 1 1" />
                 </geometry>
             </collision>
@@ -32,5 +36,5 @@
                 <origin rpy="0 0 0" xyz="0 0 0" />
                 <geometry>
-                    <mesh filename="package://simu/models/laser_robot/wheel/meshes/roda.obj" scale="1 1 1" />
+                    <mesh filename="package://robot_description/models/laser_robot/wheel/meshes/roda.obj" scale="1 1 1" />
                 </geometry>
             </visual>

File: src/simu/urdf/robot_parts/tray.xacro (robot description, xacro)
@@ -26,5 +26,5 @@
                 <origin rpy="0 0 0" xyz="0 0 0" />
                 <geometry>
-                    <mesh filename="package://simu/models/laser_robot/meshes/tray.dae" scale="1 1 1" />
+                    <mesh filename="package://robot_description/models/laser_robot/meshes/tray.dae" scale="1 1 1" />
                 </geometry>
             </collision>
@@ -32,5 +32,5 @@
                 <origin rpy="0 0 0" xyz="0 0 0" />
                 <geometry>
-                    <mesh filename="package://simu/models/laser_robot/meshes/tray.dae" scale="1 1 1" />
+                    <mesh filename="package://robot_description/models/laser_robot/meshes/tray.dae" scale="1 1 1" />
                 </geometry>
             </visual>

File: src/simu/urdf/sensors/camera.xacro (robot description, xacro)
@@ -53,5 +53,5 @@
             <origin rpy="0 0 0" xyz="0 0 0" />
             <geometry>
-                <mesh filename="package://simu/models/laser_robot/camera/meshes/camera.obj" scale="0.5 0.5 0.5" />
+                <mesh filename="package://robot_description/models/laser_robot/camera/meshes/camera.obj" scale="0.5 0.5 0.5" />
             </geometry>
         </collision>
@@ -59,5 +59,5 @@
             <origin rpy="0 0 1.57" xyz="0 0 0" />
             <geometry>
-                <mesh filename="package://simu/models/laser_robot/camera/meshes/camera.obj" scale="0.5 0.5 0.5" />
+                <mesh filename="package://robot_description/models/laser_robot/camera/meshes/camera.obj" scale="0.5 0.5 0.5" />
             </geometry>
         </visual>

File: src/simu/urdf/sensors/lidar.xacro (robot description, xacro)
@@ -50,5 +50,5 @@
       <origin rpy="0 0 0" xyz="0 0 0" />
       <geometry>
-        <mesh filename="package://simu/models/laser_robot/lidar/meshes/lidar.obj" scale="0.5 0.5 0.5" />
+        <mesh filename="package://robot_description/models/laser_robot/lidar/meshes/lidar.obj" scale="0.5 0.5 0.5" />
       </geometry>
     </collision>
@@ -56,5 +56,5 @@
       <origin rpy="0 1.57 1.57" xyz="0 0 0" />
       <geometry>
-        <mesh filename="package://simu/models/laser_robot/lidar/meshes/lidar.obj" scale="0.5 0.5 0.5" />
+        <mesh filename="package://robot_description/models/laser_robot/lidar/meshes/lidar.obj" scale="0.5 0.5 0.5" />
       </geometry>
     </visual>

File: src/simu/urdf/sensors/rplidar.xacro (robot description, xacro)
@@ -50,5 +50,5 @@
       <origin rpy="0 0 1.20" xyz="-0.03 0.02 -0.02" />
       <geometry>
-        <mesh filename="package://simu/models/laser_robot/meshes/rplidar.dae" scale="0.7 0.7 0.7" />
+        <mesh filename="package://robot_description/models/laser_robot/meshes/rplidar.dae" scale="0.7 0.7 0.7" />
       </geometry>
     </collision>
@@ -56,5 +56,5 @@
       <origin rpy="0 0 1.20" xyz="-0.03 0.02 -0.02" />
       <geometry>
-        <mesh filename="package://simu/models/laser_robot/meshes/rplidar.dae" scale="0.7 0.7 0.7" />
+        <mesh filename="package://robot_description/models/laser_robot/meshes/rplidar.dae" scale="0.7 0.7 0.7" />
       </geometry>
     </visual>

File: src/turtlebot3_description/urdf/turtlebot3_waffle.gazebo.xacro (robot description, xacro)
@@ -1,5 +1,5 @@
 <?xml version="1.0"?>
 <robot name="turtlebot3_waffle_sim" xmlns:xacro="http://ros.org/wiki/xacro">
-  <xacro:arg name="laser_visual"  default="false"/>
+  <xacro:arg name="laser_visual"  default="true"/>
   <xacro:arg name="camera_visual" default="false"/>
   <xacro:arg name="imu_visual"    default="false"/>
@@ -107,18 +107,18 @@
       <pose>0 0 0 0 0 0</pose>
       <visualize>$(arg laser_visual)</visualize>
-      <update_rate>5</update_rate>
+      <update_rate>20</update_rate>
       <ray>
         <scan>
           <horizontal>
-            <samples>360</samples>
+            <samples>${14400/20}</samples>
             <resolution>1</resolution>
-            <min_angle>0.0</min_angle>
-            <max_angle>6.28319</max_angle>
+            <min_angle>-3.14159265359</min_angle>
+            <max_angle>3.14159265359</max_angle>
           </horizontal>
         </scan>
         <range>
           <min>0.120</min>
-          <max>3.5</max>
-          <resolution>0.015</resolution>
+          <max>1.2</max>
+          <resolution>0.01</resolution>
         </range>
         <noise>
